File: hardware/Receiver/_autosave-Receiver.kicad_pcb (KiCad board)
At the start: 4 copper layers, 65 x 42 mm, 120 parts, among them J1 USB_C_Receptacle_USB2.0, J3 JST_PH, J4 Conn_01x04, Q1 2N7002, Q10 NChan, Q11 NChan, Q2 NChan, Q3 NChan, Q4 NChan, Q5 PChan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

Commit message: update mcu to ESP32S3
Connections:
- U7 pad 32: unconnected-(U7-IO36-Pad32) -> /SDA
- U7 pad 34: unconnected-(U7-IO38-Pad34) -> /SCL
Changed lines of the file:
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@@
   (net 105 "unconnected-(U7-IO8-Pad12)")
   (net 106 "unconnected-(U7-IO35-Pad31)")
-  (net 107 "unconnected-(U7-IO36-Pad32)")
-  (net 108 "unconnected-(U7-IO37-Pad33)")
-  (net 109 "unconnected-(U7-IO38-Pad34)")
-  (net 110 "unconnected-(U7-IO39{slash}TCK-Pad35)")
-  (net 111 "unconnected-(U7-IO40{slash}TDO-Pad36)")
-  (net 112 "unconnected-(U7-IO45_SPIV-Pad41)")
-  (net 113 "unconnected-(U7-IO46_DEBUGOUT-Pad44)")
-  (net 114 "/ESP_IO0")
-  (net 115 "/ESP_RX")
-  (net 116 "/ESP_TX")
+  (net 107 "unconnected-(U7-IO37-Pad33)")
+  (net 108 "unconnected-(U7-IO39{slash}TCK-Pad35)")
+  (net 109 "unconnected-(U7-IO40{slash}TDO-Pad36)")
+  (net 110 "unconnected-(U7-IO45_SPIV-Pad41)")
+  (net 111 "unconnected-(U7-IO46_DEBUGOUT-Pad44)")
+  (net 112 "/ESP_IO0")
+  (net 113 "/ESP_RX")
+  (net 114 "/ESP_TX")
   (footprint "Lipo_Charger:BQ25792" (layer "F.Cu")
     (at 132.3 89.8)
@@
       (net 51 "+3.3V") (pinfunction "3V3") (pintype "power_in") (solder_mask_margin 0.102))
     (pad "4" smd rect (at -7 -3.4 90) (size 0.8 0.4) (layers "F.Cu" "F.Paste" "F.Mask")
-      (net 114 "/ESP_IO0") (pinfunction "IO0_BOOT0") (pintype "bidirectional") (solder_mask_margin 0.102))
+      (net 112 "/ESP_IO0") (pinfunction "IO0_BOOT0") (pintype "bidirectional") (solder_mask_margin 0.102))
     (pad "5" smd rect (at -7 -2.55 90) (size 0.8 0.4) (layers "F.Cu" "F.Paste" "F.Mask")
       (net 56 "/ADDRS_LED") (pinfunction "IO1") (pintype "bidirectional") (solder_mask_margin 0.102))
@@
       (net 106 "unconnected-(U7-IO35-Pad31)") (pinfunction "IO35") (pintype "input") (solder_mask_margin 0.102))
     (pad "32" smd rect (at 7 5.1 90) (size 0.8 0.4) (layers "F.Cu" "F.Paste" "F.Mask")
-      (net 107 "unconnected-(U7-IO36-Pad32)") (pinfunction "IO36") (pintype "bidirectional") (solder_mask_margin 0.102))
+      (net 37 "/SDA") (pinfunction "IO36") (pintype "bidirectional") (solder_mask_margin 0.102))
     (pad "33" smd rect (at 7 4.25 90) (size 0.8 0.4) (layers "F.Cu" "F.Paste" "F.Mask")
-      (net 108 "unconnected-(U7-IO37-Pad33)") (pinfunction "IO37") (pintype "bidirectional") (solder_mask_margin 0.102))
+      (net 107 "unconnected-(U7-IO37-Pad33)") (pinfunction "IO37") (pintype "bidirectional") (solder_mask_margin 0.102))
     (pad "34" smd rect (at 7 3.4 90) (size 0.8 0.4) (layers "F.Cu" "F.Paste" "F.Mask")
-      (net 109 "unconnected-(U7-IO38-Pad34)") (pinfunction "IO38") (pintype "bidirectional") (solder_mask_margin 0.102))
+      (net 36 "/SCL") (pinfunction "IO38") (pintype "bidirectional") (solder_mask_margin 0.102))
     (pad "35" smd rect (at 7 2.55 90) (size 0.8 0.4) (layers "F.Cu" "F.Paste" "F.Mask")
-      (net 110 "unconnected-(U7-IO39{slash}TCK-Pad35)") (pinfunction "IO39/TCK") (pintype "bidirectional") (solder_mask_margin 0.102))
+      (net 108 "unconnected-(U7-IO39{slash}TCK-Pad35)") (pinfunction "IO39/TCK") (pintype "bidirectional") (solder_mask_margin 0.102))
     (pad "36" smd rect (at 7 1.7 90) (size 0.8 0.4) (layers "F.Cu" "F.Paste" "F.Mask")
-      (net 111 "unconnected-(U7-IO40{slash}TDO-Pad36)") (pinfunction "IO40/TDO") (pintype "bidirectional") (solder_mask_margin 0.102))
+      (net 109 "unconnected-(U7-IO40{slash}TDO-Pad36)") (pinfunction "IO40/TDO") (pintype "bidirectional") (solder_mask_margin 0.102))
     (pad "37" smd rect (at 7 0.85 90) (size 0.8 0.4) (layers "F.Cu" "F.Paste" "F.Mask")
       (net 34 "/QON") (pinfunction "IO41/TDI") (pintype "bidirectional") (solder_mask_margin 0.102))
@@
       (net 57 "/BC_INT") (pinfunction "IO42/TMS") (pintype "bidirectional") (solder_mask_margin 0.102))
     (pad "39" smd rect (at 7 -0.85 90) (size 0.8 0.4) (layers "F.Cu" "F.Paste" "F.Mask")
-      (net 116 "/ESP_TX") (pinfunction "TXD0") (pintype "bidirectional") (solder_mask_margin 0.102))
+      (net 114 "/ESP_TX") (pinfunction "TXD0") (pintype "bidirectional") (solder_mask_margin 0.102))
     (pad "40" smd rect (at 7 -1.7 90) (size 0.8 0.4) (layers "F.Cu" "F.Paste" "F.Mask")
-      (net 115 "/ESP_RX") (pinfunction "RXD0") (pintype "bidirectional") (solder_mask_margin 0.102))
+      (net 113 "/ESP_RX") (pinfunction "RXD0") (pintype "bidirectional") (solder_mask_margin 0.102))
     (pad "41" smd rect (at 7 -2.55 90) (size 0.8 0.4) (layers "F.Cu" "F.Paste" "F.Mask")
-      (net 112 "unconnected-(U7-IO45_SPIV-Pad41)") (pinfunction "IO45_SPIV") (pintype "bidirectional+no_connect") (solder_mask_margin 0.102))
+      (net 110 "unconnected-(U7-IO45_SPIV-Pad41)") (pinfunction "IO45_SPIV") (pintype "bidirectional+no_connect") (solder_mask_margin 0.102))
     (pad "42" smd rect (at 7 -3.4 90) (size 0.8 0.4) (layers "F.Cu" "F.Paste" "F.Mask")
       (net 3 "GND") (pinfunction "GND") (pintype "power_in") (solder_mask_margin 0.102))
@@
       (net 3 "GND") (pinfunction "GND") (pintype "power_in") (solder_mask_margin 0.102))
     (pad "44" smd rect (at 7 -5.1 90) (size 0.8 0.4) (layers "F.Cu" "F.Paste" "F.Mask")
-      (net 113 "unconnected-(U7-IO46_DEBUGOUT-Pad44)") (pinfunction "IO46_DEBUGOUT") (pintype "input+no_connect") (solder_mask_margin 0.102))
+      (net 111 "unconnected-(U7-IO46_DEBUGOUT-Pad44)") (pinfunction "IO46_DEBUGOUT") (pintype "input+no_connect") (solder_mask_margin 0.102))
     (pad "45" smd rect (at 7 -5.95 90) (size 0.8 0.4) (layers "F.Cu" "F.Paste" "F.Mask")
       (net 50 "/ESP_EN") (pinfunction "EN") (pintype "input") (solder_mask_margin 0.102))
@@
       (net 3 "GND") (pinfunction "1") (pintype "passive") (thermal_bridge_angle 45))
     (pad "2" smd roundrect (at -2.25 1.075 270) (size 1 0.7) (layers "F.Cu" "F.Paste" "F.Mask") (roundrect_rratio 0.25)
-      (net 114 "/ESP_IO0") (pinfunction "2") (pintype "passive") (thermal_bridge_angle 45))
+      (net 112 "/ESP_IO0") (pinfunction "2") (pintype "passive") (thermal_bridge_angle 45))
     (pad "2" smd roundrect (at 2.25 1.075 270) (size 1 0.7) (layers "F.Cu" "F.Paste" "F.Mask") (roundrect_rratio 0.25)
-      (net 114 "/ESP_IO0") (pinfunction "2") (pintype "passive") (thermal_bridge_angle 45))
+      (net 112 "/ESP_IO0") (pinfunction "2") (pintype "passive") (thermal_bridge_angle 45))
     (model "C:/Users/Andre/Documents/KiCad/7.0/3dmodels/RKB2SJK.step"
       (offset (xyz 2.2 -1.5 0))
@@
   (segment (start 176.87 113.25) (end 177.1 113.02) (width 0.254) (layer "F.Cu") (net 95))
   (segment (start 177.0375 111.75) (end 177.0375 112.9575) (width 0.254) (layer "F.Cu") (net 95))
-  (segment (start 129.125 114.15) (end 129.125 118.65) (width 0.254) (layer "F.Cu") (net 114))
-  (segment (start 127.25 111) (end 127.25 112.275) (width 0.254) (layer "F.Cu") (net 114))
-  (segment (start 127.25 112.275) (end 129.125 114.15) (width 0.254) (layer "F.Cu") (net 114))
+  (segment (start 129.125 114.15) (end 129.125 118.65) (width 0.254) (layer "F.Cu") (net 112))
+  (segment (start 127.25 111) (end 127.25 112.275) (width 0.254) (layer "F.Cu") (net 112))
+  (segment (start 127.25 112.275) (end 129.125 114.15) (width 0.254) (layer "F.Cu") (net 112))
   (zone (net 48) (net_name "/SW1") (layer "F.Cu") (hatch edge 0.5)
     (priority 15)
